File: LED_PW_HW/LED_PW_HW.kicad_pcb (KiCad board)
At the start: 2 copper layers, 44 x 44 mm, 184 parts, among them SW1 SW_MEC_5E, U1 IS31FL3732A, U2 STM32L031K6Tx, Y1 Crystal

Commit message: giving up for now and going with 72 leds
Parts:
- removed C10: 100n, Capacitor_SMD:C_0603_1608Metric_Pad1.08x0.95mm_HandSolder
- removed C11, C12, C9: 100n n.b., Capacitor_SMD:C_0603_1608Metric_Pad1.08x0.95mm_HandSolder
- removed C14, C15: 1u n.b., Capacitor_SMD:C_0603_1608Metric_Pad1.08x0.95mm_HandSolder
- removed C8: 220n n.b., Capacitor_SMD:C_0603_1608Metric_Pad1.08x0.95mm_HandSolder
- removed D100, D101, D102, D103, D104, D105, D106, D107, D108, D109, D110, D111, D112, D113, D114, D115, D116, D117, D118, D119, D120, D121, D122, D123, D124, D125, D126, D127, D128, D129, D130, D131, D132, D133, D134, D135, D136, D137, D138, D139, D140, D141, D142, D143, D144, D73, D74, D75, D76, D77, D78, D79, D80, D81, D82, D83, D84, D85, D86, D87, D88, D89, D90, D91, D92, D93, D94, D95, D96, D97, D98, D99: LED, LED_SMD:LED_0603_1608Metric_Pad1.05x0.95mm_HandSolder
- removed R10: 100k, Resistor_SMD:R_0603_1608Metric_Pad0.98x0.95mm_HandSolder
- removed TP3, TP6: TestPoint, TestPoint:TestPoint_Pad_D1.5mm
- R8: moved to B.Cu
- U1: value IS31FL3732A -> IS31FL3746A; footprint LED_PW_HW_Library:IS31FL3732A -> LED_Clock_HW:QFN-32_EP_4x4_Pitch0.4mm
- moved D65 179.5 mm to (131.8, 124.3), turned to 60 degrees
- moved D66 179.4 mm to (125.7, 118.2), turned to 30 degrees
- moved D64 179.2 mm to (140.0, 126.5), turned to 90 degrees
- moved D67 178.9 mm to (123.5, 110.0), turned to 0 degrees
- moved D63 178.6 mm to (148.2, 124.3), turned to 120 degrees
- moved D68 178.2 mm to (125.7, 101.8), turned to -30 degrees
- moved D1 178.0 mm to (160.0, 110.0)
- moved D10 178.0 mm to (151.8, 126.2)
- moved D11 178.0 mm to (150.0, 127.3)
- moved D12 178.0 mm to (148.1, 128.3)
- moved D13 178.0 mm to (146.2, 129.0)
- moved D14 178.0 mm to (144.2, 129.6)
- moved D15 178.0 mm to (142.1, 129.9)
- moved D16 178.0 mm to (140.0, 130.0)
- moved D17 178.0 mm to (137.9, 129.9)
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Connections:
- D1 pad 1: CA1 -> CS1
- D1 pad 2: CA2 -> SW1
- D10 pad 1: CA1 -> CS3
- D10 pad 2: CA3 -> SW2
- D11 pad 1: CA2 -> CS3
- D11 pad 2: CA3 -> SW3
- D12 pad 1: CA3 -> CS3
- D12 pad 2: CA2 -> SW4
- D13 pad 1: CA4 -> CS4
- D13 pad 2: CA2 -> SW1
- D14 pad 1: CA5 -> CS4
- D14 pad 2: CA2 -> SW2
- D15 pad 1: CA6 -> CS4
- D15 pad 2: CA2 -> SW3
- D16 pad 1: CA7 -> CS4
- D16 pad 2: CA2 -> SW4
- D17 pad 1: CA8 -> CS5
- D17 pad 2: CA2 -> SW1
- D18 pad 1: CA9 -> CS5
- D18 pad 2: CA2 -> SW2
- D19 pad 1: CA1 -> CS5
- D19 pad 2: CA4 -> SW3
- D2 pad 1: CA2 -> CS1
- D2 pad 2: CA1 -> SW2
- D20 pad 1: CA2 -> CS5
- D20 pad 2: CA4 -> SW4
- D21 pad 1: CA3 -> CS6
- D21 pad 2: CA4 -> SW1
- D22 pad 1: CA4 -> CS6
- D22 pad 2: CA3 -> SW2
- D23 pad 1: CA5 -> CS6
- D23 pad 2: CA3 -> SW3
- D24 pad 1: CA6 -> CS6
- D24 pad 2: CA3 -> SW4
- D25 pad 1: CA7 -> CS7
- D25 pad 2: CA3 -> SW1
- D26 pad 1: CA8 -> CS7
- D26 pad 2: CA3 -> SW2
- D27 pad 1: CA9 -> CS7
- D27 pad 2: CA3 -> SW3
- D28 pad 1: CA1 -> CS7
- D28 pad 2: CA5 -> SW4
- D29 pad 1: CA2 -> CS8
- D29 pad 2: CA5 -> SW1
- D3 pad 1: CA3 -> CS1
- D3 pad 2: CA1 -> SW3
- D30 pad 1: CA3 -> CS8
- D30 pad 2: CA5 -> SW2
- D31 pad 1: CA4 -> CS8
- D31 pad 2: CA5 -> SW3
- D32 pad 1: CA5 -> CS8
- D32 pad 2: CA4 -> SW4
- D33 pad 1: CA6 -> CS9
- D33 pad 2: CA4 -> SW1
- D34 pad 1: CA7 -> CS9
- D34 pad 2: CA4 -> SW2
- D35 pad 1: CA8 -> CS9
- D35 pad 2: CA4 -> SW3
- D36 pad 1: CA9 -> CS9
- D36 pad 2: CA4 -> SW4
- D37 pad 1: CA1 -> CS10
- D37 pad 2: CA6 -> SW1
- D38 pad 1: CA2 -> CS10
- D38 pad 2: CA6 -> SW2
- D39 pad 1: CA3 -> CS10
- D39 pad 2: CA6 -> SW3
- D4 pad 1: CA4 -> CS1
- D4 pad 2: CA1 -> SW4
- D40 pad 1: CA4 -> CS10
- D40 pad 2: CA6 -> SW4
- D41 pad 1: CA5 -> CS11
- D41 pad 2: CA6 -> SW1
- D42 pad 1: CA6 -> CS11
- D42 pad 2: CA5 -> SW2
- D43 pad 1: CA7 -> CS11
- D43 pad 2: CA5 -> SW3
- D44 pad 1: CA8 -> CS11
- D44 pad 2: CA5 -> SW4
- D45 pad 1: CA9 -> CS12
- D45 pad 2: CA5 -> SW1
- D46 pad 1: CA1 -> CS12
- D46 pad 2: CA7 -> SW2
- D47 pad 1: CA2 -> CS12
- D47 pad 2: CA7 -> SW3
- D48 pad 1: CA3 -> CS12
- D48 pad 2: CA7 -> SW4
- D49 pad 1: CA4 -> CS13
- D49 pad 2: CA7 -> SW1
- D5 pad 1: CA5 -> CS2
- D5 pad 2: CA1 -> SW1
- D50 pad 1: CA5 -> CS13
- D50 pad 2: CA7 -> SW2
- D51 pad 1: CA6 -> CS13
- D51 pad 2: CA7 -> SW3
- D52 pad 1: CA7 -> CS13
- D52 pad 2: CA6 -> SW4
- D53 pad 1: CA8 -> CS14
- D53 pad 2: CA6 -> SW1
- D54 pad 1: CA9 -> CS14
- D54 pad 2: CA6 -> SW2
- D55 pad 1: CA1 -> CS14
- D55 pad 2: CA8 -> SW3
- D56 pad 1: CA2 -> CS14
- D56 pad 2: CA8 -> SW4
- D57 pad 1: CA3 -> CS15
- D57 pad 2: CA8 -> SW1
- D58 pad 1: CA4 -> CS15
- D58 pad 2: CA8 -> SW2
- D59 pad 1: CA5 -> CS15
- D59 pad 2: CA8 -> SW3
- D6 pad 1: CA6 -> CS2
- D6 pad 2: CA1 -> SW2
- D60 pad 1: CA6 -> CS15
- D60 pad 2: CA8 -> SW4
- D61 pad 1: CA7 -> CS16
- D61 pad 2: CA8 -> SW1
- D62 pad 1: CA8 -> CS16
- D62 pad 2: CA7 -> SW2
- D63 pad 1: CA9 -> CS16
- D63 pad 2: CA7 -> SW3
- D64 pad 1: CA1 -> CS16
- D64 pad 2: CA9 -> SW4
- D65 pad 1: CA2 -> CS17
- D65 pad 2: CA9 -> SW1
- D66 pad 1: CA3 -> CS17
- D66 pad 2: CA9 -> SW2
- D67 pad 1: CA4 -> CS17
- D67 pad 2: CA9 -> SW3
- D68 pad 1: CA5 -> CS17
- D68 pad 2: CA9 -> SW4
- D69 pad 1: CA6 -> CS18
- D69 pad 2: CA9 -> SW1
- D7 pad 1: CA7 -> CS2
- D7 pad 2: CA1 -> SW3
- D70 pad 1: CA7 -> CS18
- D70 pad 2: CA9 -> SW2
- D71 pad 1: CA8 -> CS18
- D71 pad 2: CA9 -> SW3
- D72 pad 1: CA9 -> CS18
- D72 pad 2: CA8 -> SW4
- D8 pad 1: CA8 -> CS2
- D8 pad 2: CA1 -> SW4
- D9 pad 1: CA9 -> CS3
- D9 pad 2: CA1 -> SW1
- U1 pad 1: +3V3 -> CS2
- U1 pad 10: unconnected-(U1-Pad10) -> CS10
- U1 pad 11: CB1 -> CS11
- U1 pad 12: CB2 -> CS12
- U1 pad 13: CB3 -> CS13
- U1 pad 14: CB4 -> CS14
- U1 pad 15: CB5 -> CS15
- U1 pad 16: CB6 -> CS16
- U1 pad 17: CB7 -> CS17
- U1 pad 18: CB8 -> CS18
- U1 pad 19: CB9 -> +3V3
- U1 pad 2: unconnected-(U1-Pad2) -> CS3
- U1 pad 20: +3V3 -> LED_EN
- U1 pad 21: I2C_SDA -> I2C_SCL
- U1 pad 22: I2C_SCL -> GND
- U1 pad 23: GND -> I2C_SDA
- U1 pad 25: LED_EN -> SW4
- U1 pad 26: +3V3 -> SW3
- U1 pad 27: +3V3 -> SW2
- U1 pad 28: R_EXT -> SW1
- U1 pad 29: C_FILT -> +3V3
- U1 pad 3: unconnected-(U1-Pad3) -> CS4
- U1 pad 30: unconnected-(U1-Pad30) -> GND
- U1 pad 31: GND -> R_EXT
- U1 pad 32: CA1 -> CS1
- U1 pad 33: CA2 -> GND
- U1 pad 4: +3V3 -> CS5
- U1 pad 5: INTB -> CS6
- U1 pad 6: AUDIO_IN -> CS7
- U1 pad 7: GND -> CS8
- U1 pad 8: GND -> CS9
- U2 pad 18: INTB -> unconnected-(U2-Pad18)
Routing:
- net SW1: track 0.00 -> 200.1 mm, vias 0 -> 15
- net SW2: track 0.00 -> 182.1 mm, vias 0 -> 15
- net SW4: track 0.00 -> 171.3 mm, vias 0 -> 15
- net SW3: track 0.00 -> 170.8 mm, vias 0 -> 15
- net +3V3: track 0.00 -> 92.1 mm, vias 0 -> 5
- net CS15: track 0.00 -> 69.4 mm, vias 0 -> 2
- net CS14: track 0.00 -> 63.1 mm, vias 0 -> 2
- net CS13: track 0.00 -> 62.3 mm, vias 0 -> 2
- net CS17: track 0.00 -> 57.0 mm, vias 0 -> 4
- net CS12: track 0.00 -> 54.6 mm, vias 0 -> 2
- net GND: track 0.00 -> 54.2 mm, vias 0 -> 22
- net CS18: track 0.00 -> 51.8 mm, vias 0 -> 3
- net CS16: track 0.00 -> 51.2 mm, vias 0 -> 5
- net CS1: track 0.00 -> 49.4 mm, vias 0 -> 2
- net CS3: track 0.00 -> 46.3 mm, vias 0 -> 2
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- added copper zone on In2.Cu, net GND
Other:
- copper layers 2 -> 4
