File: BACKUP/v2 144 mit Treiber nd/LED_PW_HW/LED_PW_HW.kicad_pcb (KiCad board)
At the start: 4 copper layers, 44 x 44 mm, 164 parts, among them SW1 SW_MEC_5E, U2 STM32L031K6Tx, Y1 Crystal

Commit message: new version
Parts:
- added C10: 100n, Capacitor_SMD:C_0603_1608Metric_Pad1.08x0.95mm_HandSolder, F.Cu at (238.1, 154.0)
- added C11: 100n n.b., Capacitor_SMD:C_0603_1608Metric_Pad1.08x0.95mm_HandSolder, F.Cu at (252.7, 149.5)
- added C13: 1u, Capacitor_SMD:C_0603_1608Metric_Pad1.08x0.95mm_HandSolder, F.Cu at (243.0, 150.0)
- added C14: 1u n.b., Capacitor_SMD:C_0603_1608Metric_Pad1.08x0.95mm_HandSolder, F.Cu at (257.0, 152.0)
- added C15: 1u n.b., Capacitor_SMD:C_0603_1608Metric_Pad1.08x0.95mm_HandSolder, F.Cu at (257.0, 149.5)
- added C7: 100n, Capacitor_SMD:C_0603_1608Metric_Pad1.08x0.95mm_HandSolder, F.Cu at (243.0, 152.5)
- added C8: 220n n.b., Capacitor_SMD:C_0603_1608Metric_Pad1.08x0.95mm_HandSolder, F.Cu at (263.1, 83.0)
- added C9: 100n n.b., Capacitor_SMD:C_0603_1608Metric_Pad1.08x0.95mm_HandSolder, F.Cu at (252.4, 152.5)
- added R10: 100k, Resistor_SMD:R_0603_1608Metric_Pad0.98x0.95mm_HandSolder, F.Cu at (214.0, 123.0)
- added R6: 20k, Resistor_SMD:R_0603_1608Metric_Pad0.98x0.95mm_HandSolder, F.Cu at (238.1, 150.0)
- added R7: 10k, Resistor_SMD:R_0603_1608Metric_Pad0.98x0.95mm_HandSolder, F.Cu at (214.1, 130.0)
- added R8: 100k, Resistor_SMD:R_0603_1608Metric_Pad0.98x0.95mm_HandSolder, F.Cu at (214.1, 135.0)
- added R9: 10k, Resistor_SMD:R_0603_1608Metric_Pad0.98x0.95mm_HandSolder, F.Cu at (214.0, 125.5)
- added TP19: TestPoint, TestPoint:TestPoint_Pad_D1.5mm, F.Cu at (207.0, 123.0)
- added TP20: TestPoint, TestPoint:TestPoint_Pad_D1.5mm, F.Cu at (207.0, 118.0)
- added TP21: TestPoint, TestPoint:TestPoint_Pad_D1.5mm, F.Cu at (207.0, 138.0)
- added TP22: TestPoint, TestPoint:TestPoint_Pad_D1.5mm, F.Cu at (207.0, 128.0)
- added TP3: TestPoint, TestPoint:TestPoint_Pad_D1.5mm, F.Cu at (271.0, 83.0)
- added TP6: TestPoint, TestPoint:TestPoint_Pad_D1.5mm, F.Cu at (207.0, 133.0)
- added U1: IS31FL3732A, LED_PW_HW_Library:IS31FL3732A, F.Cu at (140.0, 110.0)
Connections:
- U2 pad 18: unconnected-(U2-Pad18) -> INTB
- U2 pad 19: unconnected-(U2-Pad19) -> I2C_SCL
- U2 pad 20: unconnected-(U2-Pad20) -> I2C_SDA
- U2 pad 21: unconnected-(U2-Pad21) -> I2C_PULLUP
- U2 pad 22: unconnected-(U2-Pad22) -> LED_EN
Routing:
- net CB5: track 50.4 -> 25.8 mm, vias 6 -> 0
- net CB6: track 39.8 -> 15.6 mm, vias 4 -> 0
- net CB3: track 54.0 -> 30.0 mm, vias 4 -> 0
- net +3V3: track 20.9 -> 0.00 mm
- net CB7: track 33.6 -> 16.3 mm, vias 8 -> 0
- net CB4: track 40.1 -> 22.9 mm, vias 4 -> 0
- net CB2: track 39.8 -> 24.3 mm, vias 6 -> 0
- net CB1: track 40.7 -> 25.9 mm, vias 3 -> 0
- net GND: track 13.5 -> 0.00 mm
- net CA2: track 26.8 -> 13.7 mm, vias 9 -> 0
- net CB8: track 30.7 -> 18.6 mm, vias 8 -> 0
- net CA4: track 40.2 -> 30.4 mm, vias 4 -> 0
- net CA1: track 32.6 -> 24.0 mm, vias 8 -> 0
- net CA5: track 27.6 -> 19.9 mm, vias 2 -> 0
- net CB9: track 30.5 -> 23.0 mm, vias 7 -> 0
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Other:
- board text removed: "all leds are divided into rows and columns route as much as possible on top layer then goto next one and so on (i hope i only need 2 for led routing)"
